Commit message: Align jr lidar mount with real hw

File: src/rover_sim/urdf/p3dx.urdf.xacro (robot description, xacro)
@@ -3,8 +3,7 @@
   <xacro:arg name="namespace" default="RR01" />
   <xacro:include filename="$(find rover_sim)/urdf/pioneer3dx_body.urdf.xacro" />
-  <!-- Same mount as the P3-AT model until the rover jrs' lidar is measured. -->
   <xacro:include filename="$(find ros2_livox_simulation)/urdf/mid360.xacro" />
   <xacro:mid360 name="$(arg namespace)_livox" namespace="$(arg namespace)" parent="base_link" topic="mid360" >
-    <origin xyz="0 0 0.5" rpy="0 0.349 0"/>  <!-- 0.5 m up, 20 deg down, as on the rovers -->
+    <origin xyz="0 0 0.36" rpy="0 0.524 0"/>  <!-- 0.36 m up, 30 deg down, as on the juniors -->
   </xacro:mid360>
 </robot>
