Commit message: Migrate urdfs from mighty to rover sim repo, rename ws

File: src/rover_sim/urdf/p3at.urdf.xacro (robot description, xacro)
@@ -18,5 +18,5 @@
   <xacro:arg name="namespace" default="NX01" />
   <xacro:arg name="d435_range_max_depth" default="5.0" />
-  <xacro:include filename="$(find mighty)/urdf/pioneer3at_body.urdf.xacro" />
+  <xacro:include filename="$(find rover_sim)/urdf/pioneer3at_body.urdf.xacro" />
   <!-- Disabled: fake_sim handles teleport and TF for ground robot -->
   <!-- <xacro:p3at_gazebo_ext name="$(arg namespace)_red_rover" namespace="$(arg namespace)" /> -->
@@ -26,5 +26,5 @@
   </xacro:mid360>
   <!-- Uncomment to include camera -->
-  <!-- <xacro:include filename="$(find mighty)/urdf/_d435.urdf.xacro" />
+  <!-- <xacro:include filename="$(find rover_sim)/urdf/_d435.urdf.xacro" />
   <xacro:sensor_d435 name="$(arg namespace)_d435" topics_ns="$(arg namespace)" range_max_depth="$(arg d435_range_max_depth)" parent="base_link"
                      publish_pointcloud="false" color_sensor_rate="0" depth_sensor_rate="0" depth_plugin_rate="0.0" color_plugin_rate="0.0">

File: src/rover_sim/urdf/pioneer3at_body.urdf.xacro (robot description, xacro)
@@ -24,5 +24,5 @@
 			<origin xyz="0 0 0.177" rpy="0 0 0"/>
 			<geometry name="pioneer_geom">
-				<mesh filename="package://mighty/meshes/p3at_meshes/chassis.stl"/>
+				<mesh filename="package://rover_sim/meshes/p3at/chassis.stl"/>
 			</geometry>
 			<material name="ChassisRed">
@@ -33,5 +33,5 @@
 			<origin xyz="0 0 0.177" rpy="0 0 0"/>
 				<geometry>
-					<mesh filename="package://mighty/meshes/p3at_meshes/chassis.stl"/>
+					<mesh filename="package://rover_sim/meshes/p3at/chassis.stl"/>
 				</geometry>
 		</collision>
@@ -52,5 +52,5 @@
 			<origin xyz="0 0 0" rpy="0 0 0"/>
 			<geometry name="pioneer_geom">
-				<mesh filename="package://mighty/meshes/p3at_meshes/top.stl"/>
+				<mesh filename="package://rover_sim/meshes/p3at/top.stl"/>
 			</geometry>
 			<material name="TopBlack">
@@ -78,5 +78,5 @@
 			<origin xyz="0 0 0" rpy="0 0 0"/>
 			<geometry name="pioneer_geom">
-				<mesh filename="package://mighty/meshes/p3at_meshes/front_sonar.stl"/>
+				<mesh filename="package://rover_sim/meshes/p3at/front_sonar.stl"/>
 			</geometry>
 			<material name="SonarYellow">
@@ -103,5 +103,5 @@
 			<origin xyz="0 0 0" rpy="0 0 0"/>
 			<geometry name="pioneer_geom">
-				<mesh filename="package://mighty/meshes/p3at_meshes/back_sonar.stl"/>
+				<mesh filename="package://rover_sim/meshes/p3at/back_sonar.stl"/>
 			</geometry>
 			<material name="SonarYellow">
@@ -130,5 +130,5 @@
 		<origin xyz="0 0 0" rpy="0 0 0"/>
 		<geometry name="pioneer_geom">
-			<mesh filename="package://mighty/meshes/p3at_meshes/axle.stl"/>
+			<mesh filename="package://rover_sim/meshes/p3at/axle.stl"/>
 		</geometry>
 		<material name="AxleGrey">
@@ -155,5 +155,5 @@
 		<origin xyz="0 0 0" rpy="0 0 0"/>
 		<geometry name="pioneer_geom">
-			<mesh filename="package://mighty/meshes/p3at_meshes/${side}_hubcap.stl"/>
+			<mesh filename="package://rover_sim/meshes/p3at/${side}_hubcap.stl"/>
 		</geometry>
 		<material name="HubcapYellow">
@@ -180,5 +180,5 @@
 		<origin xyz="0 0 0" rpy="0 0 0"/>
 		<geometry name="pioneer_geom">
-			<mesh filename="package://mighty/meshes/p3at_meshes/wheel.stl"/>
+			<mesh filename="package://rover_sim/meshes/p3at/wheel.stl"/>
 		</geometry>
 		<material name="WheelBlack">
@@ -189,5 +189,5 @@
 		<origin xyz="0 0 0" rpy="${-3.1415927/2} 0 0"/>
 		<geometry>
-	    <!--mesh filename="package://mighty/meshes/p3at_meshes/wheel.stl"/-->
+	    <!--mesh filename="package://rover_sim/meshes/p3at/wheel.stl"/-->
 	    <cylinder radius="0.111" length="0.075"/>
 		</geometry>
@@ -213,5 +213,5 @@
 		<origin xyz="0 0 0" rpy="0 0 0"/>
 		<geometry name="pioneer_geom">
-			<mesh filename="package://mighty/meshes/p3at_meshes/axle.stl"/>
+			<mesh filename="package://rover_sim/meshes/p3at/axle.stl"/>
 		</geometry>
 		<material name="AxleGrey">
@@ -222,5 +222,5 @@
 		<origin xyz="0 0 0" rpy="0 0 0"/>
 		<geometry>
-			<mesh filename="package://mighty/meshes/p3at_meshes/axle.stl"/>
+			<mesh filename="package://rover_sim/meshes/p3at/axle.stl"/>
 		</geometry>
 	</collision>
@@ -244,5 +244,5 @@
 		<origin xyz="0 0 0" rpy="0 0 0"/>
 		<geometry name="pioneer_geom">
-			<mesh filename="package://mighty/meshes/p3at_meshes/${side}_hubcap.stl"/>
+			<mesh filename="package://rover_sim/meshes/p3at/${side}_hubcap.stl"/>
 		</geometry>
 		<material name="HubcapYellow"/>
@@ -251,5 +251,5 @@
 		<origin xyz="0 0 0" rpy="0 0 0"/>
 		<geometry>
-			<mesh filename="package://mighty/meshes/p3at_meshes/${side}_hubcap.stl"/>
+			<mesh filename="package://rover_sim/meshes/p3at/${side}_hubcap.stl"/>
 		</geometry>
 	</collision>
@@ -274,5 +274,5 @@
 		<origin xyz="0 0 0" rpy="0 0 0"/>
 		<geometry name="pioneer_geom">
-			<mesh filename="package://mighty/meshes/p3at_meshes/wheel.stl"/>
+			<mesh filename="package://rover_sim/meshes/p3at/wheel.stl"/>
 		</geometry>
 		<material name="WheelBlack"/>
@@ -281,5 +281,5 @@
 		<origin xyz="0 0 0" rpy="${-3.1415927/2} 0 0"/>
 		<geometry>
-	    <!--mesh filename="package://mighty/meshes/p3at_meshes/wheel.stl"/-->
+	    <!--mesh filename="package://rover_sim/meshes/p3at/wheel.stl"/-->
 	    <cylinder radius="0.111" length="0.075"/>
 		</geometry>

Commit message: Align lidar mount with real hw

File: src/rover_sim/urdf/p3at.urdf.xacro (robot description, xacro)
@@ -23,5 +23,5 @@
   <xacro:include filename="$(find ros2_livox_simulation)/urdf/mid360.xacro" />
   <xacro:mid360 name="$(arg namespace)_livox" namespace="$(arg namespace)" parent="base_link" topic="mid360" >
-    <origin xyz="0 0 1.0" rpy="0 0.3 0"/>
+    <origin xyz="0 0 0.5" rpy="0 0.349 0"/>  <!-- 0.5 m up, 20 deg down, as on the rovers -->
   </xacro:mid360>
   <!-- Uncomment to include camera -->

File: src/rover_sim/urdf/p3dx.urdf.xacro (robot description, xacro)
@@ -6,5 +6,5 @@
   <xacro:include filename="$(find ros2_livox_simulation)/urdf/mid360.xacro" />
   <xacro:mid360 name="$(arg namespace)_livox" namespace="$(arg namespace)" parent="base_link" topic="mid360" >
-    <origin xyz="0 0 1.0" rpy="0 0.3 0"/>
+    <origin xyz="0 0 0.5" rpy="0 0.349 0"/>  <!-- 0.5 m up, 20 deg down, as on the rovers -->
   </xacro:mid360>
 </robot>

Commit message: Fix lidar tilt

File: src/rover_sim/urdf/p3at.urdf.xacro (robot description, xacro)
@@ -23,5 +23,5 @@
   <xacro:include filename="$(find ros2_livox_simulation)/urdf/mid360.xacro" />
   <xacro:mid360 name="$(arg namespace)_livox" namespace="$(arg namespace)" parent="base_link" topic="mid360" >
-    <origin xyz="0 0 0.5" rpy="0 0.349 0"/>  <!-- 0.5 m up, 20 deg down, as on the rovers -->
+    <origin xyz="0 0 0.5" rpy="0 0.359 0"/>  <!-- 0.5 m up, 20.6 deg down, as on the rovers -->
   </xacro:mid360>
   <!-- Uncomment to include camera -->
